File: keyboard pcb again.kicad_pcb (KiCad board)
At the start: 2 copper layers, 315.6 x 112.9 mm, 175 parts, among them J1 USB_C_Receptacle_USB2.0, J2 Conn_01x05, J3 Conn_01x04, U1 STM32F072CBT6, U2 PRTR5V0U2X, U3 XC6206PxxxMR-Regulator_Linear, U5 TXB0101

Commit message: changed to hot swap
Parts:
- removed H9: MountingHole, MountingHole:MountingHole_2.7mm_M2.5_Pad
- C1, C10, C2, C3, C4, C43, C44, C5, C6, C7, C8, C9: footprint Capacitor_SMD:C_0402_1005Metric -> Capacitor_SMD:C_1206_3216Metric
- MX1, MX10, MX11, MX12, MX13, MX14, MX15, MX16, MX17, MX18, MX19, MX2, MX20, MX21, MX22, MX23, MX24, MX25, MX26, MX27, MX28, MX29, MX3, MX30, MX31, MX32, MX33, MX34, MX35, MX36, MX37, MX38, MX39, MX4, MX40, MX41, MX42, MX43, MX44, MX45, MX46, MX47, MX48, MX49, MX5, MX50, MX51, MX52, MX53, MX54, MX55, MX56, MX57, MX58, MX59, MX6, MX60, MX61, MX62, MX63, MX64, MX65, MX66, MX67, MX68, MX69, MX7, MX8, MX9: value MX_SW_solder -> MX_SW_HS; footprint PCM_marbastlib-mx:SW_MX_1u -> PCM_marbastlib-mx:SW_MX_HS_CPG151101S11_1u
- moved J1 6.55 mm to (244.6, 302.6)
- moved C2 5.71 mm to (123.9, 393.5)
- moved D49 3.85 mm to (35.0, 374.1)
- moved D50 3.85 mm to (54.0, 374.1)
- moved D27 3.73 mm to (154.0, 336.1)
- moved D25 3.63 mm to (115.6, 336.0)
- moved D22 3.58 mm to (58.5, 335.8)
- moved D26 3.57 mm to (134.6, 335.5)
- moved D12 3.57 mm to (163.3, 316.6)
- moved D19 3.56 mm to (1.10, 335.7)
- moved D51 3.53 mm to (72.8, 374.2)
- moved D48 3.53 mm to (15.6, 374.2)
- moved D18 3.53 mm to (-17.8, 335.8)
- moved D60 3.52 mm to (-46.4, 394.2)
- moved D17 3.50 mm to (-41.6, 335.9)
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Routing:
- net GND: track 420.3 -> 357.2 mm, vias 17 -> 15
- net COL6: track 122.3 -> 88.5 mm
- net Net-(J1-CC2): track 311.2 -> 335.5 mm, vias 4 -> 6
- net COL14: track 207.2 -> 224.3 mm, vias 2 -> 4
- net COL7: track 87.0 -> 103.8 mm, vias 0 -> 4
- net Net-(D68-A): track 8.26 -> 24.0 mm
- net COL3: track 240.0 -> 251.0 mm
- net Net-(D30-A): track 8.19 -> 19.1 mm
- net Net-(D38-A): track 8.15 -> 18.9 mm
- net Net-(D28-A): track 8.01 -> 18.8 mm
- net Net-(D19-A): track 7.99 -> 18.5 mm
- net Net-(D22-A): track 7.86 -> 18.3 mm
- net Net-(D37-A): track 8.14 -> 18.5 mm
- net Net-(D15-A): track 7.97 -> 18.1 mm
- net D+: track 321.7 -> 331.7 mm
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Other:
- board size 315.6 x 112.9 mm -> 316.7 x 112.9 mm

Commit message: (should be) final pcb
Parts:
- added H9: MountingHole, MountingHole:MountingHole_2.7mm_M2.5_Pad, F.Cu at (2.98, 2.98)
- R1, R2, R3, R4: footprint Resistor_SMD:R_0402_1005Metric -> Resistor_SMD:R_1206_3216Metric
- moved R1 14.8 mm to (54.2, 388.9)
- moved R4 8.51 mm to (43.5, 390.4)
- moved U2 6.66 mm to (49.7, 388.9)
- moved R2 2.39 mm to (41.4, 387.7)
- moved D61 0.10 mm to (-27.6, 394.1)
Routing:
- net COL6: track 88.5 -> 113.8 mm, vias 2 -> 3
- net Net-(J1-CC1): track 300.8 -> 288.2 mm
- net Net-(R3-Pad2): track 1.18 -> 12.4 mm, vias 0 -> 2
- net COL11: track 213.7 -> 203.8 mm, vias 1 -> 2
- net +3V3: track 194.5 -> 203.4 mm
- net ROW2: track 334.9 -> 326.3 mm
- net +5V: track 123.2 -> 131.7 mm, vias 5 -> 6
- net COL8: track 140.3 -> 147.6 mm
- net GND: track 357.2 -> 364.4 mm
- net Net-(D68-A): track 24.0 -> 17.4 mm
- net COL7: track 103.8 -> 97.9 mm
- net COL9: track 163.9 -> 158.7 mm, vias 5 -> 2
- net Net-(D19-A): track 18.5 -> 13.7 mm
- net ROW1: track 377.1 -> 373.4 mm
- net ROW3: track 298.7 -> 295.6 mm
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
Commit message: Add files via upload
Parts:
- U5: footprint Capacitor_SMD:C_0402_1005Metric -> Capacitor_SMD:C_1206_3216Metric
- moved C44 6.31 mm to (126.6, 383.1)
Routing:
- net +5V: track 131.7 -> 136.3 mm, vias 6 -> 8
- net VBUS: track 239.6 -> 240.8 mm
- net +3V3: track 203.4 -> 202.8 mm
- net GND: track 364.4 -> 364.3 mm, vias 15 -> 16
